File: resources/project_schema/monitor_schema/esp32.sch (KiCad schematic (older format))
At the start: 19 parts, among them J2 Conn_01x03, J3 Conn_01x04, J4 Conn_01x06, J5 Conn_01x03, J6 Conn_01x03, Q1 BSS138, Q2 BSS84, SW1 SW_DPST_x2, U2 ESP32-WROOM

Commit message: Update pcb layout
Parts:
- removed SW1: SW_DPST_x2, symbol Switch:SW_DPST_x2
- added SW1, SW2: SW_MEC_5E, Button_Switch_SMD:SW_Push_1P1T_NO_6x6mm_H9.5mm, symbol Switch:SW_MEC_5E
- C3: footprint (none) -> Capacitor_SMD:C_0805_2012Metric_Pad1.18x1.45mm_HandSolder
- D1, D2: footprint (none) -> LED_SMD:LED_0805_2012Metric_Pad1.15x1.40mm_HandSolder
- J2, J5, J6: footprint (none) -> Connector_PinHeader_2.54mm:PinHeader_1x03_P2.54mm_Horizontal
- J3: footprint (none) -> Connector_PinHeader_2.54mm:PinHeader_1x04_P2.54mm_Horizontal
- J4: footprint (none) -> Connector_PinHeader_2.54mm:PinHeader_1x06_P2.54mm_Horizontal
- R1, R2, R3, R4, R5, R6, R7: footprint (none) -> Resistor_SMD:R_0805_2012Metric_Pad1.20x1.40mm_HandSolder
- U2: footprint ESP32-footprints-Lib:ESP32-WROOM -> ESPRESSIF_3DMODELS:ESP32-WROOM-32E
Connections:
- net BOOT: now also SW2.1
- net EN: now also SW1.2
- net GND: now also SW2.2
- net at C3.2, R2.2: now also SW1.1
- no-connect marks 19 -> 23
Changed lines of the file:
@@
 F 0 "R3" H 1818 5246 50  0000 L CNN
 F 1 "1k" H 1818 5155 50  0000 L CNN
-F 2 "" V 1790 5190 50  0001 C CNN
+F 2 "Resistor_SMD:R_0805_2012Metric_Pad1.20x1.40mm_HandSolder" V 1790 5190 50  0001 C CNN
 F 3 "~" H 1750 5200 50  0001 C CNN
 	1    1750 5200
@@
 F 0 "R1" H 1318 5246 50  0000 L CNN
 F 1 "1k" H 1318 5155 50  0000 L CNN
-F 2 "" V 1290 5190 50  0001 C CNN
+F 2 "Resistor_SMD:R_0805_2012Metric_Pad1.20x1.40mm_HandSolder" V 1290 5190 50  0001 C CNN
 F 3 "~" H 1250 5200 50  0001 C CNN
 	1    1250 5200
@@
 F 0 "D2" V 1789 5532 50  0000 R CNN
 F 1 "LED" V 1698 5532 50  0000 R CNN
-F 2 "" H 1750 5650 50  0001 C CNN
+F 2 "LED_SMD:LED_0805_2012Metric_Pad1.15x1.40mm_HandSolder" H 1750 5650 50  0001 C CNN
 F 3 "~" H 1750 5650 50  0001 C CNN
 	1    1750 5650
@@
 F 0 "D1" V 1289 5532 50  0000 R CNN
 F 1 "LED" V 1198 5532 50  0000 R CNN
-F 2 "" H 1250 5650 50  0001 C CNN
+F 2 "LED_SMD:LED_0805_2012Metric_Pad1.15x1.40mm_HandSolder" H 1250 5650 50  0001 C CNN
 F 3 "~" H 1250 5650 50  0001 C CNN
 	1    1250 5650
@@
 BOOT
 Wire Wire Line
-	2200 2500 2200 2650
-Connection ~ 2200 2500
-Wire Wire Line
 	2200 2500 2350 2500
 Wire Wire Line
 	2200 2350 2200 2500
-Wire Wire Line
-	2200 3050 2200 3300
-$Comp
-L Switch:SW_DPST_x2 SW?
-U 2 1 61E794C9
-P 2200 2850
-AR Path="/61E794C9" Ref="SW?"  Part="2"
-AR Path="/61E40B33/61E794C9" Ref="SW1"  Part="2"
-F 0 "SW1" V 2154 2948 50  0000 L CNN
-F 1 "SW_DPST_x2" V 2245 2948 50  0000 L CNN
-F 2 "" H 2200 2850 50  0001 C CNN
-F 3 "~" H 2200 2850 50  0001 C CNN
-	2    2200 2850
-	0    1    1    0
-$EndComp
 Text Label 1350 3250 3    50   ~ 0
 EN
-Connection ~ 1350 3100
 Wire Wire Line
 	1350 3100 1350 3250
 Connection ~ 1350 2400
-$Comp
-L Switch:SW_DPST_x2 SW?
-U 1 1 61E794D7
-P 1350 2800
-AR Path="/61E794D7" Ref="SW?"  Part="1"
-AR Path="/61E40B33/61E794D7" Ref="SW1"  Part="1"
-F 0 "SW1" V 1350 2450 50  0000 L CNN
-F 1 "SW_DPST_x2" V 1450 2300 50  0000 L CNN
-F 2 "" H 1350 2800 50  0001 C CNN
-F 3 "~" H 1350 2800 50  0001 C CNN
-	1    1350 2800
-	0    1    1    0
-$EndComp
 $Comp
 L Device:C C?
@@
 F 0 "C3" H 1585 2754 50  0000 R CNN
 F 1 "100nF" H 1585 2845 50  0000 R CNN
-F 2 "" H 1738 2650 50  0001 C CNN
+F 2 "Capacitor_SMD:C_0805_2012Metric_Pad1.18x1.45mm_HandSolder" H 1738 2650 50  0001 C CNN
 F 3 "~" H 1700 2800 50  0001 C CNN
 	1    1700 2800
 	-1   0    0    1
 $EndComp
-Wire Wire Line
-	1350 3100 1350 3000
 Wire Wire Line
 	1700 2950 1700 3100
@@
 F 0 "R4" H 2268 2246 50  0000 L CNN
 F 1 "10k" H 2268 2155 50  0000 L CNN
-F 2 "" V 2240 2190 50  0001 C CNN
+F 2 "Resistor_SMD:R_0805_2012Metric_Pad1.20x1.40mm_HandSolder" V 2240 2190 50  0001 C CNN
 F 3 "~" H 2200 2200 50  0001 C CNN
 	1    2200 2200
@@
 F 0 "U2" H 5675 3837 60  0000 C CNN
 F 1 "ESP32-WROOM" H 5675 3731 60  0000 C CNN
-F 2 "ESP32-footprints-Lib:ESP32-WROOM" H 6050 3800 60  0001 C CNN
+F 2 "ESPRESSIF_3DMODELS:ESP32-WROOM-32E" H 6050 3800 60  0001 C CNN
 F 3 "" H 5250 2900 60  0001 C CNN
 	1    5700 2450
@@
 F 0 "J2" H 9730 4492 50  0000 L CNN
 F 1 "Conn_01x03" H 9730 4401 50  0000 L CNN
-F 2 "" H 9650 4450 50  0001 C CNN
+F 2 "Connector_PinHeader_2.54mm:PinHeader_1x03_P2.54mm_Horizontal" H 9650 4450 50  0001 C CNN
 F 3 "~" H 9650 4450 50  0001 C CNN
 	1    9650 4450
@@
 F 0 "J4" H 9480 3192 50  0000 L CNN
 F 1 "Conn_01x06" H 9480 3101 50  0000 L CNN
-F 2 "" H 9400 3200 50  0001 C CNN
+F 2 "Connector_PinHeader_2.54mm:PinHeader_1x06_P2.54mm_Horizontal" H 9400 3200 50  0001 C CNN
 F 3 "~" H 9400 3200 50  0001 C CNN
 	1    9400 3200
@@
 F 0 "J3" H 9430 1592 50  0000 L CNN
 F 1 "Conn_01x04" H 9430 1501 50  0000 L CNN
-F 2 "" H 9350 1600 50  0001 C CNN
+F 2 "Connector_PinHeader_2.54mm:PinHeader_1x04_P2.54mm_Horizontal" H 9350 1600 50  0001 C CNN
 F 3 "~" H 9350 1600 50  0001 C CNN
 	1    9350 1600
@@
 Wire Wire Line
 	6600 1700 6800 1700
-Wire Wire Line
-	6600 2300 6800 2300
-Wire Wire Line
-	6600 2400 6800 2400
-Wire Wire Line
-	6600 2500 6800 2500
 Text Label 6800 2800 0    50   ~ 0
 DATA_OUT_DTH22_SENSOR
-Wire Wire Line
-	6600 2800 6800 2800
 Text Label 6800 1900 0    50   ~ 0
 RX
@@
 Wire Wire Line
 	6600 1900 6800 1900
-Wire Wire Line
-	6600 2000 6800 2000
 Text Label 6800 3100 0    50   ~ 0
 GND
@@
 Text Label 6800 2900 0    50   ~ 0
 BOOT
-Wire Wire Line
-	6600 2900 6800 2900
 Text Label 4450 1950 2    50   ~ 0
 EN
@@
 	1    0    0    -1
 $EndComp
-Wire Wire Line
-	6600 2700 6800 2700
 Wire Wire Line
 	4750 2850 4450 2850
@@
 F 0 "R5" H 3718 4896 50  0000 L CNN
 F 1 "100k" H 3718 4805 50  0000 L CNN
-F 2 "" V 3690 4840 50  0001 C CNN
+F 2 "Resistor_SMD:R_0805_2012Metric_Pad1.20x1.40mm_HandSolder" V 3690 4840 50  0001 C CNN
 F 3 "~" H 3650 4850 50  0001 C CNN
 	1    3650 4850
@@
 F 0 "R6" H 4518 5746 50  0000 L CNN
 F 1 "10k" H 4518 5655 50  0000 L CNN
-F 2 "" V 4490 5690 50  0001 C CNN
+F 2 "Resistor_SMD:R_0805_2012Metric_Pad1.20x1.40mm_HandSolder" V 4490 5690 50  0001 C CNN
 F 3 "~" H 4450 5700 50  0001 C CNN
 	1    4450 5700
@@
 F 0 "R7" H 4518 6346 50  0000 L CNN
 F 1 "10k" H 4518 6255 50  0000 L CNN
-F 2 "" V 4490 6290 50  0001 C CNN
+F 2 "Resistor_SMD:R_0805_2012Metric_Pad1.20x1.40mm_HandSolder" V 4490 6290 50  0001 C CNN
 F 3 "~" H 4450 6300 50  0001 C CNN
 	1    4450 6300
@@
 F 0 "J6" H 9730 5242 50  0000 L CNN
 F 1 "Conn_01x03" H 9730 5151 50  0000 L CNN
-F 2 "" H 9650 5200 50  0001 C CNN
+F 2 "Connector_PinHeader_2.54mm:PinHeader_1x03_P2.54mm_Horizontal" H 9650 5200 50  0001 C CNN
 F 3 "~" H 9650 5200 50  0001 C CNN
 	1    9650 5200
@@
 F 0 "J5" H 9680 5942 50  0000 L CNN
 F 1 "Conn_01x03" H 9680 5851 50  0000 L CNN
-F 2 "" H 9600 5900 50  0001 C CNN
+F 2 "Connector_PinHeader_2.54mm:PinHeader_1x03_P2.54mm_Horizontal" H 9600 5900 50  0001 C CNN
 F 3 "~" H 9600 5900 50  0001 C CNN
 	1    9600 5900
@@
 F 0 "R2" H 1418 2096 50  0000 L CNN
 F 1 "10k" H 1418 2005 50  0000 L CNN
-F 2 "" V 1390 2040 50  0001 C CNN
+F 2 "Resistor_SMD:R_0805_2012Metric_Pad1.20x1.40mm_HandSolder" V 1390 2040 50  0001 C CNN
 F 3 "~" H 1350 2050 50  0001 C CNN
 	1    1350 2050
@@
 Wire Wire Line
 	850  1100 1100 1100
+$Comp
+L Switch:SW_MEC_5E SW1
+U 1 1 61E7FFD2
+P 1250 2800
+F 0 "SW1" V 1250 2500 50  0000 L CNN
+F 1 "SW_MEC_5E" H 1050 2700 50  0000 L CNN
+F 2 "Button_Switch_SMD:SW_Push_1P1T_NO_6x6mm_H9.5mm" H 1250 3100 50  0001 C CNN
+F 3 "http://www.apem.com/int/index.php?controller=attachment&id_attachment=1371" H 1250 3100 50  0001 C CNN
+	1    1250 2800
+	0    1    1    0
+$EndComp
+$Comp
+L Switch:SW_MEC_5E SW2
+U 1 1 61E8AAE5
+P 2300 2800
+F 0 "SW2" V 2300 2500 50  0000 L CNN
+F 1 "SW_MEC_5E" H 2100 2700 50  0000 L CNN
+F 2 "Button_Switch_SMD:SW_Push_1P1T_NO_6x6mm_H9.5mm" H 2300 3100 50  0001 C CNN
+F 3 "http://www.apem.com/int/index.php?controller=attachment&id_attachment=1371" H 2300 3100 50  0001 C CNN
+	1    2300 2800
+	0    -1   1    0
+$EndComp
+NoConn ~ 2300 3000
+Wire Wire Line
+	6600 2300 6800 2300
+Wire Wire Line
+	6600 2400 6800 2400
+Wire Wire Line
+	6600 2500 6800 2500
+Wire Wire Line
+	6600 2800 6800 2800
+Wire Wire Line
+	6600 2000 6800 2000
+Wire Wire Line
+	6600 2900 6800 2900
+Wire Wire Line
+	6600 2700 6800 2700
+Connection ~ 1350 3100
+NoConn ~ 1350 3000
+Wire Wire Line
+	1100 3100 1100 2600
+Wire Wire Line
+	1100 2600 1250 2600
+Wire Wire Line
+	1100 3100 1350 3100
+NoConn ~ 1250 3000
+Wire Wire Line
+	2200 3300 2200 3150
+NoConn ~ 2200 3000
+Wire Wire Line
+	2200 3150 2450 3150
+Wire Wire Line
+	2450 3150 2450 2600
+Wire Wire Line
+	2450 2600 2300 2600
+Wire Wire Line
+	2200 2500 2200 2600
+Connection ~ 2200 2500
 $EndSCHEMATC
