File: resources/project_schema/monitor_schema/esp32.sch (KiCad schematic (older format))
At the start: 20 parts, among them J2 Conn_01x03, J3 Conn_01x04, J4 Conn_01x06, J5 Conn_01x03, J6 Conn_01x03, Q1 BSS138, Q2 BSS84, SW1 SW_MEC_5E, SW2 SW_MEC_5E, U2 ESP32-WROOM

Commit message: Change pnp transistor footprint
Parts:
- Q2: value BSS84 -> IRFL9014; footprint Package_TO_SOT_SMD:SOT-23 -> Package_TO_SOT_SMD:SOT-223
Changed lines of the file:
@@
 P 4350 5200
 F 0 "Q2" H 4554 5154 50  0000 L CNN
-F 1 "BSS84" H 4554 5245 50  0000 L CNN
-F 2 "Package_TO_SOT_SMD:SOT-23" H 4550 5125 50  0001 L CIN
+F 1 "IRFL9014" H 4554 5245 50  0000 L CNN
+F 2 "Package_TO_SOT_SMD:SOT-223" H 4550 5125 50  0001 L CIN
 F 3 "http://assets.nexperia.com/documents/data-sheet/BSS84.pdf" H 4350 5200 50  0001 L CNN
 	1    4350 5200
